File: hardware/CANx.sch (EAGLE design)
At the start: 13 parts, among them Q1 16MHz, U9 MCP2551SO8, X2 RJ45_RIGHT_ANGLEMOLEX_95001-2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, X4 RJ45_RIGHT_ANGLEMOLEX_95001-2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

Commit message: shrunk design of design to fit same enclosure as BT module
Parts:
- removed C6: 10uF, rcl:CPOL-USSMCA
- added C4: 0.1uF, rcl:C-USC0603K
- C1: value 22pF -> 10uF; device rcl:C-USC0603K -> rcl:CPOL-USSMCD
- C3: value 0.1uF -> 22pF
- renumbered C11 to C5, IC1 to U1, L2 to L1, R15 to R1, R16 to R2, U9 to U2, X4 to X1
Connections:
- net +5V: now also C1.+, C4.1; no longer C3.1, C6.+
- net GND: now also C1.-, C4.2; no longer C1.2, C6.-
- net N$2: now also C3.1; no longer C1.1
Other:
- note added: "A"
- note removed: "B"
- moved on the sheet: C3
